File: esp-buttons.sch (KiCad schematic (older format))
At the start: 41 parts, among them CON1 POWER_5V, P1 CONN_BUTTON1, P2 CONN_BUTTON2, P3 CONN_BUTTON3, P4 CONN_BUTTON4, P5 CONN_BUTTON5, P6 UART_DEBUG, P7 UART, P8 POWER_5V, P9 USB_B, Q1 IRLML2502TRPBF, Q2 IRLML2502TRPBF, Q3 IRLML2502TRPBF, Q4 IRLML2502TRPBF, Q5 IRLML2502TRPBF, SW1 RESET_BUTTON, SW2 PROG_BUTTON, U1 ESP-07v2, U2 LD1117S33CTR, U3 FT230XS

Commit message: Modified the switches sch symbols to have only 2 pin on the schematic
Parts:
- P2: footprint Terminal_Blocks:TerminalBlock_Pheonix_PT-3.5mm_2pol -> Terminal_Blocks:TerminalBlock_Pheonix_PT-3.5mm_4pol
- P9: value USB_B -> USB
- SW1, SW2: symbol Switch_DPST -> SW_PUSH
Connections:
- net GND: no longer SW1.4, SW2.4
- net PROG: no longer SW2.3
- net RESET: now also R8.2, U1.3 (CH_PD); no longer SW1.3
Other:
- moved on the sheet: R10
Changed lines of the file:
@@
 U 1 1 57C6C352
 P 1000 1050
-F 0 "CON1" H 1000 1300 50  0000 C CNN
-F 1 "POWER_5V" H 1000 850 50  0000 C CNN
+F 0 "CON1" H 750 1300 50  0000 C CNN
+F 1 "POWER_5V" H 850 850 50  0000 C CNN
 F 2 "Connect:JACK_ALIM" H 1000 1050 50  0001 C CNN
 F 3 "" H 1000 1050 50  0000 C CNN
@@
 $EndComp
 $Comp
-L Switch_DPST SW1
+L SW_PUSH SW1
 U 1 1 57C6D3AF
-P 5000 2150
-F 0 "SW1" V 4600 2050 50  0000 C CNN
-F 1 "RESET_BUTTON" V 5400 2050 50  0000 C CNN
-F 2 "Buttons_Switches_ThroughHole:SW_PUSH_6mm" H 5000 2150 50  0001 C CNN
-F 3 "" H 5000 2150 50  0000 C CNN
-	1    5000 2150
-	0    1    1    0
+P 5200 2250
+F 0 "SW1" V 4950 2350 50  0000 C CNN
+F 1 "RESET_BUTTON" V 5450 2550 50  0000 C CNN
+F 2 "Buttons_Switches_ThroughHole:SW_PUSH_6mm" H 5200 2250 50  0001 C CNN
+F 3 "" H 5200 2250 50  0000 C CNN
+	1    5200 2250
+	0    -1   1    0
 $EndComp
 $Comp
@@
 L R_Small R10
 U 1 1 57C83F0C
-P 9800 2750
-F 0 "R10" H 9600 2800 50  0000 L CNN
-F 1 "10K" H 9600 2700 50  0000 L CNN
-F 2 "Resistors_SMD:R_1206_HandSoldering" H 9800 2750 50  0001 C CNN
-F 3 "" H 9800 2750 50  0000 C CNN
-	1    9800 2750
+P 10000 2750
+F 0 "R10" H 9800 2800 50  0000 L CNN
+F 1 "10K" H 9800 2700 50  0000 L CNN
+F 2 "Resistors_SMD:R_1206_HandSoldering" H 10000 2750 50  0001 C CNN
+F 3 "" H 10000 2750 50  0000 C CNN
+	1    10000 2750
 	-1   0    0    -1
 $EndComp
@@
 L +3V3 #PWR013
 U 1 1 57C83F12
-P 9800 2600
-F 0 "#PWR013" H 9800 2450 50  0001 C CNN
-F 1 "+3V3" H 9800 2740 50  0000 C CNN
-F 2 "" H 9800 2600 50  0000 C CNN
-F 3 "" H 9800 2600 50  0000 C CNN
-	1    9800 2600
-	-1   0    0    -1
-$EndComp
-$Comp
-L Switch_DPST SW2
+P 10000 2600
+F 0 "#PWR013" H 10000 2450 50  0001 C CNN
+F 1 "+3V3" H 10000 2740 50  0000 C CNN
+F 2 "" H 10000 2600 50  0000 C CNN
+F 3 "" H 10000 2600 50  0000 C CNN
+	1    10000 2600
+	-1   0    0    -1
+$EndComp
+$Comp
+L SW_PUSH SW2
 U 1 1 57C83F19
-P 10000 3250
-F 0 "SW2" V 9600 3050 50  0000 C CNN
-F 1 "PROG_BUTTON" V 10400 3150 50  0000 C CNN
-F 2 "Buttons_Switches_ThroughHole:SW_PUSH_6mm" H 10000 3250 50  0001 C CNN
-F 3 "" H 10000 3250 50  0000 C CNN
-	1    10000 3250
-	0    -1   1    0
+P 10000 3300
+F 0 "SW2" V 9750 3400 50  0000 C CNN
+F 1 "PROG_BUTTON" V 10250 3600 50  0000 C CNN
+F 2 "Buttons_Switches_ThroughHole:SW_PUSH_6mm" H 10000 3300 50  0001 C CNN
+F 3 "" H 10000 3300 50  0000 C CNN
+	1    10000 3300
+	0    1    1    0
 $EndComp
 Text Label 7850 2250 0    60   ~ 0
@@
 F 0 "P2" H 600 4650 50  0000 C CNN
 F 1 "CONN_BUTTON2" H 350 4150 50  0000 C CNN
-F 2 "Terminal_Blocks:TerminalBlock_Pheonix_PT-3.5mm_2pol" H 600 4400 50  0001 C CNN
+F 2 "Terminal_Blocks:TerminalBlock_Pheonix_PT-3.5mm_4pol" H 600 4400 50  0001 C CNN
 F 3 "" H 600 4400 50  0000 C CNN
 	1    600  4400
@@
 P 10050 5050
 F 0 "P9" V 9750 4950 50  0000 C CNN
-F 1 "USB_B" V 10250 4950 50  0000 C CNN
+F 1 "USB" V 10250 4950 50  0000 C CNN
 F 2 "Connect:USB_B" V 10000 4950 50  0001 C CNN
 F 3 "" V 10000 4950 50  0000 C CNN
@@
 	5200 1300 5200 1450
 Wire Wire Line
-	5200 1850 5200 1650
+	5200 1650 5200 1950
 Wire Wire Line
 	7850 2150 9050 2150
@@
 	7850 2350 8550 2350
 Wire Wire Line
-	9800 2600 9800 2650
-Wire Wire Line
-	9800 2950 9800 2850
-Wire Wire Line
-	9800 3550 9800 3800
+	10000 2600 10000 2650
 Wire Wire Line
 	8850 2950 8850 2250
@@
 	4450 6400 4450 6600
 Wire Wire Line
-	5600 2050 5600 1650
+	5600 1650 5600 2050
 Wire Wire Line
 	8350 4950 9750 4950
@@
 L GND #PWR028
 U 1 1 57E98CE4
-P 9800 3800
-F 0 "#PWR028" H 9800 3550 50  0001 C CNN
-F 1 "GND" H 9800 3650 50  0000 C CNN
-F 2 "" H 9800 3800 50  0000 C CNN
-F 3 "" H 9800 3800 50  0000 C CNN
-	1    9800 3800
-	1    0    0    -1
-$EndComp
-Wire Wire Line
-	10200 3550 9800 3550
-Wire Wire Line
-	8850 2950 10200 2950
-Connection ~ 9800 2950
-Wire Wire Line
-	4800 1850 6050 1850
-Connection ~ 5200 1850
-Wire Wire Line
-	4800 2450 5200 2450
-Wire Wire Line
-	5200 2450 5200 2650
+P 10000 3650
+F 0 "#PWR028" H 10000 3400 50  0001 C CNN
+F 1 "GND" H 10000 3500 50  0000 C CNN
+F 2 "" H 10000 3650 50  0000 C CNN
+F 3 "" H 10000 3650 50  0000 C CNN
+	1    10000 3650
+	1    0    0    -1
+$EndComp
 Wire Wire Line
 	3700 5900 3700 5550
 Wire Wire Line
-	3700 6650 3700 6550
+	3700 6550 3700 6650
 Wire Wire Line
 	4450 6600 3700 6600
@@
 	1    0    0    -1
 $EndComp
+Wire Wire Line
+	5200 1850 6050 1850
+Connection ~ 5600 1850
+Connection ~ 5200 1850
+Wire Wire Line
+	5200 2550 5200 2650
+Wire Wire Line
+	10000 3650 10000 3600
+Wire Wire Line
+	10000 2850 10000 3000
+Wire Wire Line
+	8850 2950 10000 2950
+Connection ~ 10000 2950
 $EndSCHEMATC
